File: Gotek.kicad_pcb (KiCad board)
At the start: 2 copper layers, 111.6 x 59.4 mm, 72 parts, among them J10 Conn_01x04_Pin, J3 Conn_01x03_Pin, J4 Conn_01x02_Pin, J7 Display Port, P1 Conn_01x26, P3 USB_A, Q1 PMBT2222A,215, Q2 PMBT2222A,215, Q3 PMBT2222A,215, Q4 PMBT2222A,215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

Commit message: Add files via upload
Corrected values for R10 and RN13 (4K7).
Parts:
- R10, RN13: value 1K -> 4K7
Changed lines of the file:
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@@
 			)
 		)
-		(property "Value" "1K"
+		(property "Value" "4K7"
 			(at 0 1.65 90)
 			(layer "F.Fab")
@@
 			)
 		)
-		(property "Value" "1K"
+		(property "Value" "4K7"
 			(at 0 1.65 0)
 			(layer "F.Fab")
